Commit message: Align URDF joint convention with bhl_arm_1

File: urdf/lite_000_asm.urdf (robot description, URDF)
Before this commit: robot lite_000_asm, 114 links, 113 joints
Links:
- added link left_gripper_tip_middle_link, mass 1e-9
- added link right_gripper_tip_middle_link, mass 1e-9
Joints:
- added joint left_gripper_tip_middle_joint: type fixed, parent left_gripper_slider_base_link, child left_gripper_tip_middle_link, origin xyz=-0.0743543 0 0.0047 rpy=0 0 0
- added joint right_gripper_tip_middle_joint: type fixed, parent right_gripper_slider_base_link, child right_gripper_tip_middle_link, origin xyz=-0.0749871 0 0.0047 rpy=0 0 0
- joint left_elbow_pitch_joint: limit lower=-0.182318 upper=2.17388 effort=1 velocity=1 -> lower=-2.356198 upper=0 effort=1 velocity=1; origin xyz=0 0 -0.001 rpy=-3.14159 0 3.14159 -> xyz=0 0 -0.001 rpy=-3.14159 0.0000005 2.959272
- joint left_shoulder_pitch_joint: limit lower=-1.8997 upper=2.02729 effort=1 velocity=1 -> lower=-3.1415916 upper=0.7853984 effort=1 velocity=1; origin xyz=0 0 -0.004 rpy=0 -1.5708 4.71239 -> xyz=0 0 -0.004 rpy=2.0272911 -1.5707927 1.5707973
- joint left_shoulder_roll_joint: axis 0 -1 0 -> 0 1 0; limit lower=-3.00182 upper=0.488835 effort=1 velocity=1 -> lower=-0.1745326 upper=3.3161224 effort=1 velocity=1; origin xyz=0 0 -0.001 rpy=-1.5708 0 3.14159 -> xyz=0 0 -0.001 rpy=-1.5707998 0.0000011 -2.8272929
- joint left_shoulder_yaw_joint: limit lower=-1.13098 upper=2.01062 effort=1 velocity=1 -> lower=-1.5708 upper=1.5708 effort=1 velocity=1; origin xyz=0.013435 -0.013435 -0.052 rpy=0 -1.5708 4.71239 -> xyz=0.013435 -0.013435 -0.052 rpy=-2.7017727 -1.5707927 1.5707973
- joint left_wrist_pitch_joint: axis 0 0 -1 -> 0 0 1; limit lower=-1.24937 upper=0.32143 effort=1 velocity=1 -> lower=-0.7854 upper=0.7854 effort=1 velocity=1; origin xyz=0 0 0 rpy=0 1.5708 1.5708 -> xyz=0 0 0 rpy=1.5708045 1.1068263 -3.1415816
- joint left_wrist_roll_joint: limit lower=-1.11223 upper=0.284037 effort=1 velocity=1 -> lower=-0.6981335 upper=0.6981335 effort=1 velocity=1; origin xyz=-0.137 -0.026 0 rpy=0 0 0 -> xyz=-0.137 -0.026 0 rpy=0 0.4140965 0
- joint left_wrist_yaw_joint: limit lower=-3.04023 upper=0.101359 effort=1 velocity=1 -> lower=-1.5707945 upper=1.5707945 effort=1 velocity=1; origin xyz=-0.0339087 -0.0551924 -0.0271 rpy=3.14159 0.101359 2.43568 -> xyz=-0.0339087 -0.0551924 -0.0271 rpy=2.1761163 1.5707931 1.4702039
- joint right_elbow_pitch_joint: limit lower=-1.87973 upper=0.476469 effort=1 velocity=1 -> lower=-2.356199 upper=0 effort=1 velocity=1; origin xyz=0 0 -0.001 rpy=3.14159 0 -1.5708 -> xyz=0 0 -0.001 rpy=3.1415903 0.0000012 -1.094331
- joint right_shoulder_pitch_joint: limit lower=-2.72505 upper=1.20194 effort=1 velocity=1 -> lower=-3.1415916 upper=0.7853984 effort=1 velocity=1; origin xyz=0 0 -0.004 rpy=0 1.5708 1.5708 -> xyz=0 0 -0.004 rpy=2.7250511 1.5707927 -1.5707927
- joint right_shoulder_roll_joint: limit lower=-0.756945 upper=2.73371 effort=1 velocity=1 -> lower=-3.3161224 upper=0.1745326 effort=1 velocity=1; origin xyz=-0.013435 -0.013435 -0.052 rpy=-1.5708 0 3.14159 -> xyz=-0.013435 -0.013435 -0.052 rpy=-1.5707994 -0.000002 2.5591776
- joint right_shoulder_yaw_joint: limit lower=-3.12357 upper=0.0180244 effort=1 velocity=1 -> lower=-1.5707972 upper=1.5707972 effort=1 velocity=1; origin xyz=0 0 -0.052 rpy=0 1.5708 -1.5708 -> xyz=0 0 -0.052 rpy=-1.5888199 1.5707927 1.5707927
- joint right_wrist_pitch_joint: axis 0 0 -1 -> 0 0 1; limit lower=-1.03932 upper=0.531478 effort=1 velocity=1 -> lower=-0.785399 upper=0.785399 effort=1 velocity=1; origin xyz=0 0 0 rpy=0 1.5708 -4.71239 -> xyz=0 0 0 rpy=1.5708109 1.3168753 -3.1415795
- joint right_wrist_roll_joint: axis 0 -1 0 -> 0 1 0; limit lower=-0.623811 upper=0.772453 effort=1 velocity=1 -> lower=-0.698132 upper=0.698132 effort=1 velocity=1; origin xyz=0.137 -0.026 0 rpy=0 0 0 -> xyz=0.137 -0.026 0 rpy=0 -0.074321 0
- joint right_wrist_yaw_joint: limit lower=-0.556921 upper=2.58467 effort=1 velocity=1 -> lower=-1.5707955 upper=1.5707955 effort=1 velocity=1; origin xyz=0.0634578 -0.0130041 -0.0264 rpy=3.14159 1.01388 -1.61793 -> xyz=0.0634578 -0.0130041 -0.0264 rpy=3.1415913 0.0000055 -1.6179277

Commit message: Tune gripper midpoint task frames

File: urdf/lite_000_asm.urdf (robot description, URDF)
Before this commit: robot lite_000_asm, 116 links, 115 joints
Joints:
- joint left_gripper_tip_middle_joint: origin xyz=-0.0743543 0 0.0047 rpy=0 0 0 -> xyz=-0.0743543 0 0.063 rpy=0 0 0
- joint right_gripper_tip_middle_joint: origin xyz=-0.0749871 0 0.0047 rpy=0 0 0 -> xyz=-0.0749871 0 0.063 rpy=0 0 0
