Commit message: Refine gripper controls and collision geometry
Expose one control joint per gripper and keep the opposite finger as a passive mimic joint.

Sync collision primitives with the latest URDF export and normalize gripper lower-limit initialization, including the corrected left gripper closed pose.

Update RL handoff notes, README, and CAD name mappings for the new gripper interface.

File: urdf/lite_arm_gripper.urdf (robot description, URDF)
Before this commit: robot lite_000_asm, 116 links, 115 joints
Links:
- link chest_link: geometry collision cylinder length=0.209443 radius=0.054721; visual mesh filename=package://lite_urdf/meshes/chest_body.stl
- link left_gripper_finger_left_link: geometry visual mesh filename=package://lite_urdf/meshes/gripper_left_finger.stl
- link left_gripper_finger_right_link: geometry visual mesh filename=package://lite_urdf/meshes/gripper_right_finger.stl
- link left_gripper_palm_link: geometry collision box size=0.038 0.042 0.06; visual mesh filename=package://lite_urdf/meshes/gripper_palm.stl
- link left_gripper_rack_base_link: geometry collision cylinder length=0.18 radius=0.005; visual mesh filename=package://lite_urdf/meshes/gripper_rack_base.stl
- link left_gripper_rack_mount_link: geometry collision box size=0.038 0.042 0.06; visual mesh filename=package://lite_urdf/meshes/gripper_rack_mount.stl
- link right_gripper_palm_link: geometry collision box size=0.038 0.042 0.06; visual mesh filename=package://lite_urdf/meshes/gripper_palm.stl
- link right_gripper_rack_base_link: geometry collision cylinder length=0.18 radius=0.005; visual mesh filename=package://lite_urdf/meshes/gripper_rack_base.stl
- link right_gripper_rack_mount_link: geometry collision box size=0.038 0.042 0.06; visual mesh filename=package://lite_urdf/meshes/gripper_rack_mount.stl
Joints:
- removed joint left_gripper_left_finger_joint
- removed joint left_gripper_right_finger_joint
- removed joint right_gripper_left_finger_joint
- removed joint right_gripper_right_finger_joint
- added joint left_gripper_joint: type prismatic, parent left_gripper_slider_base_link, child left_gripper_finger_left_link, origin xyz=-0.03975 0.0035 0.0033 rpy=0 0 0, axis 1 0 0, limit lower=0 upper=0.047 effort=1 velocity=1
- added joint left_gripper_passive_joint: type prismatic, parent left_gripper_slider_base_link, child left_gripper_finger_right_link, origin xyz=-0.11025 0.0035 0.0033 rpy=0 0 0, axis -1 0 0, limit lower=0 upper=0.047 effort=1 velocity=1, mimic joint=left_gripper_joint multiplier=1 offset=0
- added joint right_gripper_joint: type prismatic, parent right_gripper_slider_base_link, child right_gripper_finger_left_link, origin xyz=-0.0397241 0.0035 0.0033 rpy=0 0 0, axis 1 0 0, limit lower=0 upper=0.047 effort=1 velocity=1
- added joint right_gripper_passive_joint: type prismatic, parent right_gripper_slider_base_link, child right_gripper_finger_right_link, origin xyz=-0.11025 0.0035 0.0033 rpy=0 0 0, axis -1 0 0, limit lower=0 upper=0.047 effort=1 velocity=1, mimic joint=right_gripper_joint multiplier=1 offset=0
- joint left_elbow_pitch_joint: axis 0 0 -1 -> 0 0 1
- joint left_shoulder_pitch_joint: axis 1 0 0 -> -1 0 0
- joint right_shoulder_roll_joint: axis 0 -1 0 -> 0 1 0

Commit message: Use fixed-link merged STL URDF

File: urdf/lite_arm_gripper.urdf (robot description, URDF)
Before this commit: robot lite_000_asm, 116 links, 115 joints
Links:
- removed link base_support_beam_link
- removed link base_support_link
- removed link base_vertical_link
- removed link body_front_plate_link
- removed link body_rear_panel_link
- removed link body_top_disc_assembly_link
- removed link body_top_disc_link
- removed link body_top_plate_link
- removed link chest_base_mount_link
- removed link chest_connector_left_link
- removed link chest_connector_right_link
- removed link chest_link
- removed link frame_assembly_link
- removed link frame_back_left_short_link
- removed link frame_back_left_upright_link
- removed link frame_back_right_short_link
- removed link frame_back_right_upright_link
- removed link frame_center_rail_link
- removed link frame_front_left_rail_link
- removed link frame_front_left_short_link
- removed link frame_front_left_upright_link
- removed link frame_front_right_rail_link
- removed link frame_front_right_short_link
- removed link frame_front_right_upright_link
- removed link frame_left_side_rail_link
- removed link frame_rail_assembly_link
- removed link frame_right_side_rail_link
- removed link frame_spine_link
- removed link head_camera_optical_frame
- removed link left_elbow_actuator_link
- removed link left_elbow_pitch_cover_link
- removed link left_gripper_actuator_link
- removed link left_gripper_lower_rack_link
- removed link left_gripper_palm_link
- removed link left_gripper_rack_base_link
- removed link left_gripper_rack_mount_link
- removed link left_gripper_rack_strut_link
- removed link left_gripper_slider_base_link
- removed link left_gripper_upper_rack_link
- removed link left_shoulder_base_link
- removed link left_shoulder_pitch_cover_link
- removed link left_shoulder_pitch_motor_link
- removed link left_shoulder_roll_actuator_link
- removed link left_shoulder_roll_cover_link
- removed link left_shoulder_yaw_actuator_link
- removed link left_shoulder_yaw_cover_link
- removed link left_shoulder_yaw_limit_link
- removed link left_wrist_breakout_board_link
- removed link left_wrist_camera_cad_link
- removed link left_wrist_camera_mount_body_link
- removed link left_wrist_camera_mount_link
- removed link left_wrist_camera_mount_plate_link
- removed link left_wrist_camera_optical_frame
- removed link left_wrist_horn_link
- removed link left_wrist_pitch_cover_link
- removed link left_wrist_roll_aux_motor_link
- removed link left_wrist_roll_motor_link
- removed link left_wrist_yaw_aux_motor_link
- removed link left_wrist_yaw_cover_link
- removed link left_wrist_yaw_link
- removed link right_elbow_actuator_link
- removed link right_elbow_pitch_cover_link
- removed link right_gripper_actuator_link
- removed link right_gripper_lower_rack_link
- removed link right_gripper_palm_link
- removed link right_gripper_rack_base_link
- removed link right_gripper_rack_mount_link
- removed link right_gripper_rack_strut_link
- removed link right_gripper_slider_base_link
- removed link right_gripper_upper_rack_link
- removed link right_shoulder_base_link
- removed link right_shoulder_pitch_aux_link
- removed link right_shoulder_pitch_cover_link
- removed link right_shoulder_pitch_motor_link
- removed link right_shoulder_roll_actuator_link
- removed link right_shoulder_roll_cover_link
- removed link right_shoulder_yaw_actuator_link
- removed link right_shoulder_yaw_aux_link
- removed link right_shoulder_yaw_cover_link
- removed link right_shoulder_yaw_limit_link
- removed link right_wrist_camera_cad_link
- removed link right_wrist_camera_mount_body_link
- removed link right_wrist_camera_mount_link
- removed link right_wrist_camera_mount_plate_link
- removed link right_wrist_camera_optical_frame
- removed link right_wrist_horn_link
- removed link right_wrist_pitch_cover_link
- removed link right_wrist_roll_aux_motor_link
- removed link right_wrist_roll_link
- removed link right_wrist_yaw_aux_motor_link
- removed link right_wrist_yaw_cover_link
- removed link right_wrist_yaw_link
- link left_elbow_pitch_link: geometry visual mesh filename=package://lite_urdf/meshes/left_elbow_pitch_link_visual.stl
- link left_gripper_finger_left_link: geometry collision mesh filename=package://lite_urdf/meshes/left_gripper_finger_left_link_co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; visual mesh filename=package://lite_urdf/meshes/left_gripper_finger_left_link_vi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
- link left_gripper_finger_right_link: geometry collision mesh filename=package://lite_urdf/meshes/left_gripper_finger_right_link_c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; visual mesh filename=package://lite_urdf/meshes/left_gripper_finger_right_link_v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
- link left_shoulder_pitch_link: geometry collision cylinder length=0.06 radius=0.03; visual mesh filename=package://lite_urdf/meshes/left_shoulder_pitch_link_visual.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
- link left_shoulder_roll_link: geometry collision cylinder length=0.1 radius=0.03; visual mesh filename=package://lite_urdf/meshes/left_shoulder_roll_link_visual.s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
- link left_shoulder_yaw_link: geometry collision cylinder length=0.06 radius=0.03; visual mesh filename=package://lite_urdf/meshes/left_shoulder_yaw_link_visual.stl
- link left_wrist_pitch_link: geometry collision box size=0.04 0.04 0.01; collision cylinder length=0.04 radius=0.023
- link left_wrist_roll_link: geometry collision cylinder length=0.045 radius=0.026; visual mesh filename=package://lite_urdf/meshes/left_wrist_roll_link_visual.stl
- link left_wrist_yaw_motor_link: geometry collision cylinder length=0.12 radius=0.03; visual mesh filename=package://lite_urdf/meshes/left_wrist_yaw_motor_link_visual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
- link right_elbow_pitch_link: geometry visual mesh filename=package://lite_urdf/meshes/right_elbow_pitch_link_visual.stl
- link right_gripper_finger_left_link: geometry collision mesh filename=package://lite_urdf/meshes/right_gripper_finger_left_link_c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; visual mesh filename=package://lite_urdf/meshes/right_gripper_finger_left_link_v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
- link right_gripper_finger_right_link: geometry collision mesh filename=package://lite_urdf/meshes/right_gripper_finger_right_link_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; visual mesh filename=package://lite_urdf/meshes/right_gripper_finger_right_link_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
- link right_shoulder_pitch_link: geometry collision cylinder length=0.06 radius=0.03; visual mesh filename=package://lite_urdf/meshes/right_shoulder_pitch_link_visual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
- link right_shoulder_roll_link: geometry collision cylinder length=0.1 radius=0.03; visual mesh filename=package://lite_urdf/meshes/right_shoulder_roll_link_visual.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
- link right_shoulder_yaw_link: geometry collision cylinder length=0.06 radius=0.03; visual mesh filename=package://lite_urdf/meshes/right_shoulder_yaw_link_visual.s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
- link right_wrist_pitch_link: geometry collision box size=0.04 0.04 0.01; collision cylinder length=0.04 radius=0.023
- link right_wrist_roll_motor_link: geometry collision cylinder length=0.045002 radius=0.026; visual mesh filename=package://lite_urdf/meshes/right_wrist_roll_motor_link_visu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
- link right_wrist_yaw_motor_link: geometry collision cylinder length=0.12 radius=0.03; visual mesh filename=package://lite_urdf/meshes/right_wrist_yaw_motor_link_visua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
- link world_root: geometry collision cylinder length=0.209443 radius=0.054721; visual mesh filename=package://lite_urdf/meshes/world_root_visual.stl
Joints:
- removed joint chest_connector_left_joint
- removed joint chest_connector_right_joint
- removed joint fixed_10_joint
- removed joint fixed_11_joint
- removed joint fixed_12_joint
- removed joint fixed_13_joint
- removed joint fixed_14_joint
- removed joint fixed_1_10_joint
- removed joint fixed_1_11_joint
- removed joint fixed_1_12_joint
- removed joint fixed_1_13_joint
- removed joint fixed_1_14_joint
- removed joint fixed_1_15_joint
- removed joint fixed_1_16_joint
- removed joint fixed_1_17_joint
- removed joint fixed_1_18_joint
- removed joint fixed_1_19_joint
- removed joint fixed_1_1_joint
- removed joint fixed_1_20_joint
- removed joint fixed_1_21_joint
- removed joint fixed_1_22_joint
- removed joint fixed_1_23_joint
- removed joint fixed_1_2_joint
- removed joint fixed_1_3_joint
- removed joint fixed_1_4_joint
- removed joint fixed_1_5_joint
- removed joint fixed_1_6_joint
- removed joint fixed_1_7_joint
- removed joint fixed_1_8_joint
- removed joint fixed_1_9_joint
- removed joint fixed_1_joint
- removed joint fixed_2_10_joint
- removed joint fixed_2_11_joint
- removed joint fixed_2_12_joint
- removed joint fixed_2_13_joint
- removed joint fixed_2_14_joint
- removed joint fixed_2_15_joint
- removed joint fixed_2_16_joint
- removed joint fixed_2_17_joint
- removed joint fixed_2_18_joint
- removed joint fixed_2_19_joint
- removed joint fixed_2_1_joint
- removed joint fixed_2_20_joint
- removed joint fixed_2_2_joint
- removed joint fixed_2_3_joint
- removed joint fixed_2_4_joint
- removed joint fixed_2_5_joint
- removed joint fixed_2_6_joint
- removed joint fixed_2_7_joint
- removed joint fixed_2_8_joint
- removed joint fixed_2_9_joint
- removed joint fixed_2_joint
- removed joint fixed_3_10_joint
- removed joint fixed_3_11_joint
- removed joint fixed_3_12_joint
- removed joint fixed_3_13_joint
- removed joint fixed_3_14_joint
- removed joint fixed_3_1_joint
- removed joint fixed_3_2_joint
- removed joint fixed_3_3_joint
- removed joint fixed_3_4_joint
- removed joint fixed_3_5_joint
- removed joint fixed_3_6_joint
- removed joint fixed_3_7_joint
- removed joint fixed_3_8_joint
- removed joint fixed_3_9_joint
- removed joint fixed_3_joint
- removed joint fixed_4_1_joint
- removed joint fixed_4_2_joint
- removed joint fixed_4_3_joint
- removed joint fixed_4_4_joint
- removed joint fixed_4_5_joint
- removed joint fixed_4_joint
- removed joint fixed_5_1_joint
- removed joint fixed_5_2_joint
- removed joint fixed_5_3_joint
- removed joint fixed_5_joint
- removed joint fixed_6_1_joint
- removed joint fixed_6_2_joint
- removed joint fixed_6_joint
- removed joint fixed_7_1_joint
- removed joint fixed_7_2_joint
- removed joint fixed_7_joint
- removed joint fixed_8_1_joint
- removed joint fixed_8_2_joint
- removed joint fixed_8_joint
- removed joint fixed_9_joint
- removed joint frame_assembly_to_frame_rail_assembly_joint
- removed joint head_camera_optical_joint
- removed joint left_wrist_camera_optical_joint
- removed joint right_wrist_camera_optical_joint
- removed joint world_root_to_base_vertical_joint
- joint head_camera_joint: origin xyz=0 0.10828 0.28 rpy=0 0.7853982 1.5707963 -> xyz=-1.937121605e-06 -0.1082753717 1.010000795 rpy=0 0.7853908536 -1.570796354; parent chest_link -> world_root
- joint left_elbow_pitch_joint: origin xyz=0 0 -0.001 rpy=-3.14159 0.0000005 2.959272 -> xyz=-0.0800000025 0.02048037438 0.02003692937 rpy=-0.2962759628 -0.3299797087 -0.8151948384; parent left_elbow_actuator_link -> left_shoulder_yaw_link
- joint left_gripper_joint: origin xyz=-0.03975 0.0035 0.0033 rpy=0 0 0 -> xyz=0.1040961904 -0.04585909073 -0.01258790935 rpy=1.5708 -0.0698132 0.845028; parent left_gripper_slider_base_link -> left_wrist_pitch_link
- joint left_gripper_passive_joint: origin xyz=-0.11025 0.0035 0.0033 rpy=0 0 0 -> xyz=0.05741859357 -0.09846390861 -0.01750574286 rpy=1.5708 -0.0698132 0.845028; parent left_gripper_slider_base_link -> left_wrist_pitch_link
- joint left_gripper_tip_middle_joint: origin xyz=-0.0743543 0 0.063 rpy=0 0 0 -> xyz=0.1260019346 -0.1111205665 -0.01849347726 rpy=1.5708 -0.0698132 0.845028; parent left_gripper_slider_base_link -> left_wrist_pitch_link
- joint left_shoulder_pitch_joint: origin xyz=0 0 -0.004 rpy=2.0272911 -1.5707927 1.5707973 -> xyz=0.04962222198 -0.007996932602 0.7928799915 rpy=0.2994274351 0.1745330072 -3.141587582; parent left_shoulder_pitch_motor_link -> world_root
- joint left_shoulder_roll_joint: origin xyz=0 0 -0.001 rpy=-1.5707998 0.0000011 -2.8272929 -> xyz=-0.04100000351 0.02565540881 -0.007919662552 rpy=-0.7846655169 1.140163396 -0.7368651954; parent left_shoulder_roll_actuator_link -> left_shoulder_pitch_link
- joint left_shoulder_yaw_joint: origin xyz=0.013435 -0.013435 -0.052 rpy=-2.7017727 -1.5707927 1.5707973 -> xyz=0.1148822482 -0.02709980309 -0.03734592284 rpy=-2.701771727 -0.3143027 -3.14158898; parent left_shoulder_yaw_actuator_link -> left_shoulder_roll_link
- joint left_wrist_camera_joint: origin xyz=0 0 0 rpy=0 0 0 -> xyz=0.1237537251 -0.1140010331 0.02440096001 rpy=-0.785393176 -0.06981242277 0.845026119; parent left_wrist_camera_cad_link -> left_wrist_pitch_link
- joint left_wrist_pitch_joint: origin xyz=0 0 0 rpy=1.5708045 1.1068263 -3.1415816 -> xyz=-0.009053135665 0.026 0.02059831873 rpy=0.2838290718 0.30570169 -2.371804821; parent left_wrist_roll_aux_motor_link -> left_wrist_roll_link
- joint left_wrist_roll_joint: origin xyz=-0.137 -0.026 0 rpy=0 0.4140965 0 -> xyz=-0.02599949677 -0.1370000955 -6.899333461e-08 rpy=3.141589755 -0.4140965 1.570801166; parent left_wrist_yaw_link -> left_wrist_yaw_motor_link
- joint right_elbow_pitch_joint: origin xyz=0 0 -0.001 rpy=3.1415903 0.0000012 -1.094331 -> xyz=0.08000000295 0.0270258376 -0.009514478403 rpy=-1.552756021 0.04712209601 0.0008482378368; parent right_elbow_actuator_link -> right_shoulder_yaw_link
- joint right_gripper_joint: origin xyz=-0.0397241 0.0035 0.0033 rpy=0 0 0 -> xyz=0.113421574 -0.009254971529 -0.01265282701 rpy=1.5708 -0.0698132 1.17725; parent right_gripper_slider_base_link -> right_wrist_pitch_link
- joint right_gripper_passive_joint: origin xyz=-0.11025 0.0035 0.0033 rpy=0 0 0 -> xyz=0.08644316447 -0.07423085268 -0.0175724672 rpy=1.5708 -0.0698132 1.17725; parent right_gripper_slider_base_link -> right_wrist_pitch_link
- joint right_gripper_tip_middle_joint: origin xyz=-0.0749871 0 0.063 rpy=0 0 0 -> xyz=0.1551621984 -0.06441037825 -0.01860434352 rpy=1.5708 -0.0698132 1.17725; parent right_gripper_slider_base_link -> right_wrist_pitch_link
- joint right_shoulder_pitch_joint: origin xyz=0 0 -0.004 rpy=2.7250511 1.5707927 -1.5707927 -> xyz=-0.04962609453 -0.007796944815 0.7928799997 rpy=-0.2594571717 -0.1745330458 3.141587621; parent right_shoulder_pitch_motor_link -> world_root
- joint right_shoulder_roll_joint: origin xyz=-0.013435 -0.013435 -0.052 rpy=-1.5707994 -0.000002 2.5591776 -> xyz=0.04099980899 0.02527477392 0.006709218258 rpy=2.691965127 0.9393656487 2.770140483; parent right_shoulder_roll_actuator_link -> right_shoulder_pitch_link
- joint right_shoulder_yaw_joint: origin xyz=0 0 -0.052 rpy=-1.5888199 1.5707927 1.5707927 -> xyz=0.1008846481 -0.02639984048 0.06644494687 rpy=1.55277638 -0.5824100464 3.673220854e-06; parent right_shoulder_yaw_actuator_link -> right_shoulder_roll_link
- joint right_wrist_camera_joint: origin xyz=0 0 0 rpy=0 0 0 -> xyz=0.1542184407 -0.06728357609 0.02433415705 rpy=-0.7853878688 -0.06981242277 1.177248119; parent right_wrist_camera_cad_link -> right_wrist_pitch_link
- joint right_wrist_pitch_joint: origin xyz=0 0 0 rpy=1.5708109 1.3168753 -3.1415795 -> xyz=0.0016707 0.026 0.0224379 rpy=0.02854527272 0.06862962747 0.3945277653; parent right_wrist_roll_aux_motor_link -> right_wrist_roll_motor_link
- joint right_wrist_roll_joint: origin xyz=0.137 -0.026 0 rpy=0 -0.074321 0 -> xyz=-4.077257665e-07 -0.137 -0.026 rpy=1.57079999 2.727450251e-07 -1.645121; parent right_wrist_yaw_link -> right_wrist_yaw_motor_link
- joint right_wrist_yaw_joint: origin xyz=0.0634578 -0.0130041 -0.0264 rpy=3.1415913 0.0000055 -1.6179277 -> xyz=0.0634578 -0.0130041 -0.0264 rpy=3.1415913 5.5e-06 -1.6179277
