Commit message: Add GoldenGlow visuals and headless URDF

File: urdf/lite_arm_gripper_headless.urdf (robot description, URDF)
Before this commit: robot lite_000_asm, 24 links, 23 joints
Links:
- removed link head_camera_link
- link world_root: geometry collision cylinder length=0.209443 radius=0.054721; visual mesh filename=package://lite_urdf/meshes/world_root_headless.stl
Joints:
- removed joint head_camera_joint
