Commit message: Fix O6 hand wrist roll joints

File: urdf/lite_flash_arm_hand.urdf (robot description, URDF)
Before this commit: robot lite_flash_arm_hand, 44 links, 43 joints
Joints:
- joint lh_wrist_roll: axis 0 0 1 -> (none); limit lower=-3.141592653589793 upper=3.141592653589793 effort=10 velocity=3.14 -> (none); origin xyz=0 0 0 rpy=0 0 0 -> xyz=0 0 0 rpy=0 0 1.5707963268; type revolute -> fixed
- joint rh_wrist_roll: axis 0 0 1 -> (none); limit lower=-3.141592653589793 upper=3.141592653589793 effort=10 velocity=3.14 -> (none); origin xyz=0 0 0 rpy=0 0 0 -> xyz=0 0 0 rpy=0 0 -1.5707963268; type revolute -> fixed

File: urdf/lite_pro_arm_hand.urdf (robot description, URDF)
Before this commit: robot lite_pro_arm_hand, 44 links, 43 joints
Joints:
- joint lh_wrist_roll: axis 0 0 1 -> (none); limit lower=-3.141592653589793 upper=3.141592653589793 effort=10 velocity=3.14 -> (none); origin xyz=0 0 0 rpy=0 0 0 -> xyz=0 0 0 rpy=0 0 1.5707963268; type revolute -> fixed
- joint rh_wrist_roll: axis 0 0 1 -> (none); limit lower=-3.141592653589793 upper=3.141592653589793 effort=10 velocity=3.14 -> (none); origin xyz=0 0 0 rpy=0 0 0 -> xyz=0 0 0 rpy=0 0 -1.5707963268; type revolute -> fixed
