Commit message: Add headless O6 hand URDF variants

File: urdf/lite_flash_arm_hand_headless.urdf (robot description, URDF)
Before this commit: robot lite_flash_arm_hand, 42 links, 41 joints
Links:
- link world_root: geometry collision cylinder length=0.209443 radius=0.054721; visual mesh filename=package://lite_urdf/meshes/world_root_headless.stl

File: urdf/lite_pro_arm_hand.urdf (robot description, URDF)
Before this commit: robot lite_pro_arm_hand, 44 links, 43 joints
Links:
- removed link left_wrist_camera_link
- removed link right_wrist_camera_link
Joints:
- removed joint left_wrist_camera_joint
- removed joint right_wrist_camera_joint

File: urdf/lite_pro_arm_hand_headless.urdf (robot description, URDF)
Before this commit: robot lite_flash_arm_hand, 42 links, 41 joints
Links:
- link left_elbow_pitch_link: geometry collision mesh filename=package://lite_urdf/meshes/left_elbow_pitch_link_visual.stl; visual mesh filename=package://lite_urdf/meshes/left_elbow_pitch_link_visual.stl
- link left_shoulder_pitch_link: geometry collision mesh filename=package://lite_urdf/meshes/left_shoulder_pitch_link_visual.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; visual mesh filename=package://lite_urdf/meshes/left_shoulder_pitch_link_visual.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
- link left_shoulder_roll_link: geometry collision mesh filename=package://lite_urdf/meshes/left_shoulder_roll_link_visual.s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; visual mesh filename=package://lite_urdf/meshes/left_shoulder_roll_link_visual.s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
- link left_shoulder_yaw_link: geometry collision mesh filename=package://lite_urdf/meshes/left_shoulder_yaw_link_visual.stl; visual mesh filename=package://lite_urdf/meshes/left_shoulder_yaw_link_visual.stl
- link left_wrist_roll_link: geometry collision mesh filename=package://lite_urdf/meshes/left_wrist_roll_link_visual.stl; visual mesh filename=package://lite_urdf/meshes/left_wrist_roll_link_visual.stl
- link left_wrist_yaw_motor_link: geometry collision mesh filename=package://lite_urdf/meshes/left_wrist_yaw_motor_link_visual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; visual mesh filename=package://lite_urdf/meshes/left_wrist_yaw_motor_link_visual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
- link right_elbow_pitch_link: geometry collision mesh filename=package://lite_urdf/meshes/right_elbow_pitch_link_visual.stl; visual mesh filename=package://lite_urdf/meshes/right_elbow_pitch_link_visual.stl
- link right_shoulder_pitch_link: geometry collision mesh filename=package://lite_urdf/meshes/right_shoulder_pitch_link_visual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; visual mesh filename=package://lite_urdf/meshes/right_shoulder_pitch_link_visual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
- link right_shoulder_roll_link: geometry collision mesh filename=package://lite_urdf/meshes/right_shoulder_roll_link_visual.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; visual mesh filename=package://lite_urdf/meshes/right_shoulder_roll_link_visual.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
- link right_shoulder_yaw_link: geometry collision mesh filename=package://lite_urdf/meshes/right_shoulder_yaw_link_visual.s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; visual mesh filename=package://lite_urdf/meshes/right_shoulder_yaw_link_visual.s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
- link right_wrist_roll_motor_link: geometry collision mesh filename=package://lite_urdf/meshes/right_wrist_roll_motor_link_visu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; visual mesh filename=package://lite_urdf/meshes/right_wrist_roll_motor_link_visu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
- link right_wrist_yaw_motor_link: geometry collision mesh filename=package://lite_urdf/meshes/right_wrist_yaw_motor_link_visua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; visual mesh filename=package://lite_urdf/meshes/right_wrist_yaw_motor_link_visua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
- link world_root: geometry collision mesh filename=package://lite_urdf/meshes/world_root_headless.stl; visual mesh filename=package://lite_urdf/meshes/world_root_headless.stl
