Commit message: fix: correct all camera frame orientation

File: urdf/lite_flash_arm_gripper.urdf (robot description, URDF)
Before this commit: robot lite_000_asm, 24 links, 23 joints
Joints:
- joint head_camera_joint: origin xyz=-1.937121605e-06 -0.1082753717 1.010000795 rpy=0 0.7853908536 -1.570796354 -> xyz=-1.937121605e-06 -0.1082753717 1.010000795 rpy=-2.3561871804 0 3.1415926264
- joint left_wrist_camera_joint: origin xyz=0.1237537251 -0.1140010331 0.02440096001 rpy=-0.785393176 -0.06981242277 0.845026119 -> xyz=0.1237537251 -0.1140010331 0.02440096001 rpy=-2.3561994776 0.0698124228 -2.2965665346
- joint right_wrist_camera_joint: origin xyz=0.1542184407 -0.06728357609 0.02433415705 rpy=-0.7853878688 -0.06981242277 1.177248119 -> xyz=0.1542184407 -0.06728357609 0.02433415705 rpy=-2.3562047848 0.0698124228 -1.9643445346

File: urdf/lite_flash_arm_gripper_headless.urdf (robot description, URDF)
Before this commit: robot lite_000_asm_headless, 23 links, 22 joints
Links:
- added link head_camera_link, mass 1e-9
Joints:
- added joint head_camera_joint: type fixed, parent world_root, child head_camera_link, origin xyz=-1.937121605e-06 -0.1082753717 1.010000795 rpy=-2.3561871804 0 3.1415926264
- joint left_wrist_camera_joint: origin xyz=0.1237537251 -0.1140010331 0.02440096001 rpy=-0.785393176 -0.06981242277 0.845026119 -> xyz=0.1237537251 -0.1140010331 0.02440096001 rpy=-2.3561994776 0.0698124228 -2.2965665346
- joint right_wrist_camera_joint: origin xyz=0.1542184407 -0.06728357609 0.02433415705 rpy=-0.7853878688 -0.06981242277 1.177248119 -> xyz=0.1542184407 -0.06728357609 0.02433415705 rpy=-2.3562047848 0.0698124228 -1.9643445346

File: urdf/lite_pro_arm_gripper.urdf (robot description, URDF)
Before this commit: robot lite_000_asm, 24 links, 23 joints
Joints:
- joint head_camera_joint: origin xyz=-1.937121605e-06 -0.1082753717 1.010000795 rpy=0 0.7853908536 -1.570796354 -> xyz=-1.937121605e-06 -0.1082753717 1.010000795 rpy=-2.3561871804 0 3.1415926264
- joint left_wrist_camera_joint: origin xyz=0.1237537251 -0.1140010331 0.02440096001 rpy=-0.785393176 -0.06981242277 0.845026119 -> xyz=0.1237537251 -0.1140010331 0.02440096001 rpy=-2.3561994776 0.0698124228 -2.2965665346
- joint right_wrist_camera_joint: origin xyz=0.1542184407 -0.06728357609 0.02433415705 rpy=-0.7853878688 -0.06981242277 1.177248119 -> xyz=0.1542184407 -0.06728357609 0.02433415705 rpy=-2.3562047848 0.0698124228 -1.9643445346

File: urdf/lite_pro_arm_gripper_headless.urdf (robot description, URDF)
Before this commit: robot lite_000_asm_headless, 23 links, 22 joints
Links:
- added link head_camera_link, mass 1e-9
Joints:
- added joint head_camera_joint: type fixed, parent world_root, child head_camera_link, origin xyz=-1.937121605e-06 -0.1082753717 1.010000795 rpy=-2.3561871804 0 3.1415926264
- joint left_wrist_camera_joint: origin xyz=0.1237537251 -0.1140010331 0.02440096001 rpy=-0.785393176 -0.06981242277 0.845026119 -> xyz=0.1237537251 -0.1140010331 0.02440096001 rpy=-2.3561994776 0.0698124228 -2.2965665346
- joint right_wrist_camera_joint: origin xyz=0.1542184407 -0.06728357609 0.02433415705 rpy=-0.7853878688 -0.06981242277 1.177248119 -> xyz=0.1542184407 -0.06728357609 0.02433415705 rpy=-2.3562047848 0.0698124228 -1.9643445346

Commit message: feat!: update Lite URDF joint convention and EVA theme
Align shoulder-roll zero pose with bar_description_lite/lite_ros2, fold RL handoff notes into the README, remove the installed config docs directory, and update visual materials to the EVA-inspired palette.

BREAKING CHANGE: Shoulder-roll zero pose and limits are shifted relative to the previous bhl_arm_1-compatible URDF convention.

File: urdf/lite_flash_arm_gripper.urdf (robot description, URDF)
Before this commit: robot lite_000_asm, 24 links, 23 joints
Joints:
- joint left_shoulder_roll_joint: limit lower=-0.1745326 upper=3.3161224 effort=1 velocity=1 -> lower=-1.57079475 upper=1.91986025 effort=1 velocity=1; origin xyz=-0.04100000351 0.02565540881 -0.007919662552 rpy=-0.7846655169 1.140163396 -0.7368651954 -> xyz=-0.04100000351 0.02565540881 -0.007919662552 rpy=-2.8052323666 0.4653133292 -2.9859660904
- joint right_shoulder_roll_joint: limit lower=-3.3161224 upper=0.1745326 effort=1 velocity=1 -> lower=-1.91986025 upper=1.57079475 effort=1 velocity=1; origin xyz=0.04099980899 0.02527477392 0.006709218258 rpy=2.691965127 0.9393656487 2.770140483 -> xyz=0.04099980899 0.02527477392 0.006709218258 rpy=0.3501154544 0.7257811284 0.2377861735

File: urdf/lite_flash_arm_gripper_headless.urdf (robot description, URDF)
Before this commit: robot lite_000_asm_headless, 24 links, 23 joints
Joints:
- joint left_shoulder_roll_joint: limit lower=-0.1745326 upper=3.3161224 effort=1 velocity=1 -> lower=-1.57079475 upper=1.91986025 effort=1 velocity=1; origin xyz=-0.04100000351 0.02565540881 -0.007919662552 rpy=-0.7846655169 1.140163396 -0.7368651954 -> xyz=-0.04100000351 0.02565540881 -0.007919662552 rpy=-2.8052323666 0.4653133292 -2.9859660904
- joint right_shoulder_roll_joint: limit lower=-3.3161224 upper=0.1745326 effort=1 velocity=1 -> lower=-1.91986025 upper=1.57079475 effort=1 velocity=1; origin xyz=0.04099980899 0.02527477392 0.006709218258 rpy=2.691965127 0.9393656487 2.770140483 -> xyz=0.04099980899 0.02527477392 0.006709218258 rpy=0.3501154544 0.7257811284 0.2377861735

File: urdf/lite_flash_arm_hand.urdf (robot description, URDF)
Before this commit: robot lite_flash_arm_hand, 42 links, 41 joints
Joints:
- joint left_shoulder_roll_joint: limit lower=-0.1745326 upper=3.3161224 effort=1 velocity=1 -> lower=-1.57079475 upper=1.91986025 effort=1 velocity=1; origin xyz=-0.04100000351 0.02565540881 -0.007919662552 rpy=-0.7846655169 1.140163396 -0.7368651954 -> xyz=-0.04100000351 0.02565540881 -0.007919662552 rpy=-2.8052323666 0.4653133292 -2.9859660904
- joint right_shoulder_roll_joint: limit lower=-3.3161224 upper=0.1745326 effort=1 velocity=1 -> lower=-1.91986025 upper=1.57079475 effort=1 velocity=1; origin xyz=0.04099980899 0.02527477392 0.006709218258 rpy=2.691965127 0.9393656487 2.770140483 -> xyz=0.04099980899 0.02527477392 0.006709218258 rpy=0.3501154544 0.7257811284 0.2377861735

File: urdf/lite_flash_arm_hand_headless.urdf (robot description, URDF)
Before this commit: robot lite_flash_arm_hand_headless, 42 links, 41 joints
Joints:
- joint left_shoulder_roll_joint: limit lower=-0.1745326 upper=3.3161224 effort=1 velocity=1 -> lower=-1.57079475 upper=1.91986025 effort=1 velocity=1; origin xyz=-0.04100000351 0.02565540881 -0.007919662552 rpy=-0.7846655169 1.140163396 -0.7368651954 -> xyz=-0.04100000351 0.02565540881 -0.007919662552 rpy=-2.8052323666 0.4653133292 -2.9859660904
- joint right_shoulder_roll_joint: limit lower=-3.3161224 upper=0.1745326 effort=1 velocity=1 -> lower=-1.91986025 upper=1.57079475 effort=1 velocity=1; origin xyz=0.04099980899 0.02527477392 0.006709218258 rpy=2.691965127 0.9393656487 2.770140483 -> xyz=0.04099980899 0.02527477392 0.006709218258 rpy=0.3501154544 0.7257811284 0.2377861735

File: urdf/lite_pro_arm_gripper.urdf (robot description, URDF)
Before this commit: robot lite_000_asm, 24 links, 23 joints
Joints:
- joint left_shoulder_roll_joint: limit lower=-0.1745326 upper=3.3161224 effort=1 velocity=1 -> lower=-1.57079475 upper=1.91986025 effort=1 velocity=1; origin xyz=-0.04100000351 0.02565540881 -0.007919662552 rpy=-0.7846655169 1.140163396 -0.7368651954 -> xyz=-0.04100000351 0.02565540881 -0.007919662552 rpy=-2.8052323666 0.4653133292 -2.9859660904
- joint right_shoulder_roll_joint: limit lower=-3.3161224 upper=0.1745326 effort=1 velocity=1 -> lower=-1.91986025 upper=1.57079475 effort=1 velocity=1; origin xyz=0.04099980899 0.02527477392 0.006709218258 rpy=2.691965127 0.9393656487 2.770140483 -> xyz=0.04099980899 0.02527477392 0.006709218258 rpy=0.3501154544 0.7257811284 0.2377861735

File: urdf/lite_pro_arm_gripper_headless.urdf (robot description, URDF)
Before this commit: robot lite_000_asm_headless, 24 links, 23 joints
Joints:
- joint left_shoulder_roll_joint: limit lower=-0.1745326 upper=3.3161224 effort=1 velocity=1 -> lower=-1.57079475 upper=1.91986025 effort=1 velocity=1; origin xyz=-0.04100000351 0.02565540881 -0.007919662552 rpy=-0.7846655169 1.140163396 -0.7368651954 -> xyz=-0.04100000351 0.02565540881 -0.007919662552 rpy=-2.8052323666 0.4653133292 -2.9859660904
- joint right_shoulder_roll_joint: limit lower=-3.3161224 upper=0.1745326 effort=1 velocity=1 -> lower=-1.91986025 upper=1.57079475 effort=1 velocity=1; origin xyz=0.04099980899 0.02527477392 0.006709218258 rpy=2.691965127 0.9393656487 2.770140483 -> xyz=0.04099980899 0.02527477392 0.006709218258 rpy=0.3501154544 0.7257811284 0.2377861735

File: urdf/lite_pro_arm_hand.urdf (robot description, URDF)
Before this commit: robot lite_pro_arm_hand, 42 links, 41 joints
Joints:
- joint left_shoulder_roll_joint: limit lower=-0.1745326 upper=3.3161224 effort=1 velocity=1 -> lower=-1.57079475 upper=1.91986025 effort=1 velocity=1; origin xyz=-0.04100000351 0.02565540881 -0.007919662552 rpy=-0.7846655169 1.140163396 -0.7368651954 -> xyz=-0.04100000351 0.02565540881 -0.007919662552 rpy=-2.8052323666 0.4653133292 -2.9859660904
- joint right_shoulder_roll_joint: limit lower=-3.3161224 upper=0.1745326 effort=1 velocity=1 -> lower=-1.91986025 upper=1.57079475 effort=1 velocity=1; origin xyz=0.04099980899 0.02527477392 0.006709218258 rpy=2.691965127 0.9393656487 2.770140483 -> xyz=0.04099980899 0.02527477392 0.006709218258 rpy=0.3501154544 0.7257811284 0.2377861735

File: urdf/lite_pro_arm_hand_headless.urdf (robot description, URDF)
Before this commit: robot lite_pro_arm_hand_headless, 42 links, 41 joints
Joints:
- joint left_shoulder_roll_joint: limit lower=-0.1745326 upper=3.3161224 effort=1 velocity=1 -> lower=-1.57079475 upper=1.91986025 effort=1 velocity=1; origin xyz=-0.04100000351 0.02565540881 -0.007919662552 rpy=-0.7846655169 1.140163396 -0.7368651954 -> xyz=-0.04100000351 0.02565540881 -0.007919662552 rpy=-2.8052323666 0.4653133292 -2.9859660904
- joint right_shoulder_roll_joint: limit lower=-3.3161224 upper=0.1745326 effort=1 velocity=1 -> lower=-1.91986025 upper=1.57079475 effort=1 velocity=1; origin xyz=0.04099980899 0.02527477392 0.006709218258 rpy=2.691965127 0.9393656487 2.770140483 -> xyz=0.04099980899 0.02527477392 0.006709218258 rpy=0.3501154544 0.7257811284 0.2377861735
