Commit message: feat: prepare Lite URDF for ROS 2 production integration

File: urdf/lite.urdf.xacro (robot description, xacro)
@@ -1,4 +1,17 @@
 <?xml version='1.0' encoding='utf-8'?>
-<robot name="lite_000_asm_headless">
+<robot xmlns:xacro="http://www.ros.org/wiki/xacro" name="lite_000_asm">
+    <!--
+      Xacro source for the checked-in URDF variant. Joint/link transforms and
+      mesh frames are preserved from lite_urdf; exposed arm/gripper joint names
+      and optional ros2_control metadata follow lite_urdf.
+    -->
+    <xacro:arg name="emit_ros2_control" default="true"/>
+    <xacro:arg name="use_fake_hardware" default="true"/>
+    <xacro:arg name="use_sim" default="false"/>
+    <xacro:arg name="mode" default="arms_grippers"/>
+    <xacro:arg name="can_interface_left" default="can0"/>
+    <xacro:arg name="can_interface_right" default="can1"/>
+    <xacro:arg name="calibration_file" default=""/>
+    <xacro:include filename="lite.ros2_control.xacro"/>
     <link name="right_wrist_yaw_motor_link">
         <inertial>
@@ -418,5 +431,5 @@
             <origin xyz="0 0 0" rpy="0 0 0" />
             <geometry>
-                <mesh filename="package://lite_urdf/meshes/world_root_headless.stl" />
+                <mesh filename="package://lite_urdf/meshes/world_root_visual.stl" />
             </geometry>
             <material name="lite_world_root">
@@ -466,5 +479,77 @@
         </inertial>
     </link>
-    <joint name="left_wrist_pitch_joint" type="revolute">
+    <joint name="left_shoulder_pitch" type="revolute">
+        <parent link="world_root" />
+        <child link="left_shoulder_pitch_link" />
+        <origin xyz="0.04962222198 -0.007996932602 0.7928799915" rpy="0.2994274351 0.1745330072 -3.141587582" />
+        <axis xyz="-1 0 0" />
+        <limit lower="-3.1415916" upper="0.7853984" effort="1" velocity="1" />
+        <hardware>
+            <motorType>None</motorType>
+            <motorDirection>-1</motorDirection>
+            <armature>0</armature>
+        </hardware>
+    </joint>
+    <joint name="left_shoulder_roll" type="revolute">
+        <parent link="left_shoulder_pitch_link" />
+        <child link="left_shoulder_roll_link" />
+        <origin xyz="-0.04100000351 0.02565540881 -0.007919662552" rpy="-2.8052323666 0.4653133292 -2.9859660904" />
+        <axis xyz="0 1 0" />
+        <limit lower="-1.57079475" upper="1.91986025" effort="1" velocity="1" />
+        <hardware>
+            <motorType>None</motorType>
+            <motorDirection>-1</motorDirection>
+            <armature>0</armature>
+        </hardware>
+    </joint>
+    <joint name="left_shoulder_yaw" type="revolute">
+        <parent link="left_shoulder_roll_link" />
+        <child link="left_shoulder_yaw_link" />
+        <origin xyz="0.1148822482 -0.02709980309 -0.03734592284" rpy="-2.701771727 -0.3143027 -3.14158898" />
+        <axis xyz="1 0 0" />
+        <limit lower="-1.5708" upper="1.5708" effort="1" velocity="1" />
+        <hardware>
+            <motorType>None</motorType>
+            <motorDirection>1</motorDirection>
+            <armature>0</armature>
+        </hardware>
+    </joint>
+    <joint name="left_elbow_pitch" type="revolute">
+        <parent link="left_shoulder_yaw_link" />
+        <child link="left_elbow_pitch_link" />
+        <origin xyz="-0.0800000025 0.02048037438 0.02003692937" rpy="-0.2962759628 -0.3299797087 -0.8151948384" />
+        <axis xyz="0 0 1" />
+        <limit lower="-2.356198" upper="0" effort="1" velocity="1" />
+        <hardware>
+            <motorType>None</motorType>
+            <motorDirection>-1</motorDirection>
+            <armature>0</armature>
+        </hardware>
+    </joint>
+    <joint name="left_wrist_yaw" type="revolute">
+        <parent link="left_elbow_pitch_link" />
+        <child link="left_wrist_yaw_motor_link" />
+        <origin xyz="-0.0339087 -0.0551924 -0.0271" rpy="2.1761163 1.5707931 1.4702039" />
+        <axis xyz="0 1 0" />
+        <limit lower="-1.5707945" upper="1.5707945" effort="1" velocity="1" />
+        <hardware>
+            <motorType>None</motorType>
+            <motorDirection>1</motorDirection>
+            <armature>0</armature>
+        </hardware>
+    </joint>
+    <joint name="left_wrist_roll" type="revolute">
+        <parent link="left_wrist_yaw_motor_link" />
+        <child link="left_wrist_roll_link" />
+        <origin xyz="-0.02599949677 -0.1370000955 -6.899333461e-08" rpy="3.141589755 -0.4140965 1.570801166" />
+        <axis xyz="0 -1 0" />
+        <limit lower="-0.6981335" upper="0.6981335" effort="1" velocity="1" />
+        <hardware>
+            <motorType>None</motorType>
+            <motorDirection>-1</motorDirection>
+            <armature>0</armature>
+        </hardware>
+    </joint>
+    <joint name="left_wrist_pitch" type="revolute">
         <parent link="left_wrist_roll_link" />
         <child link="left_wrist_pitch_link" />
@@ -474,72 +559,12 @@
         <hardware>
             <motorType>None</motorType>
-            <motorDirection>1</motorDirection>
-            <armature>0</armature>
-        </hardware>
-    </joint>
-    <joint name="left_wrist_roll_joint" type="revolute">
-        <parent link="left_wrist_yaw_motor_link" />
-        <child link="left_wrist_roll_link" />
-        <origin xyz="-0.02599949677 -0.1370000955 -6.899333461e-08" rpy="3.141589755 -0.4140965 1.570801166" />
-        <axis xyz="0 -1 0" />
-        <limit lower="-0.6981335" upper="0.6981335" effort="1" velocity="1" />
-        <hardware>
-            <motorType>None</motorType>
-            <motorDirection>1</motorDirection>
-            <armature>0</armature>
-        </hardware>
-    </joint>
-    <joint name="left_wrist_yaw_joint" type="revolute">
-        <parent link="left_elbow_pitch_link" />
-        <child link="left_wrist_yaw_motor_link" />
-        <origin xyz="-0.0339087 -0.0551924 -0.0271" rpy="2.1761163 1.5707931 1.4702039" />
-        <axis xyz="0 1 0" />
-        <limit lower="-1.5707945" upper="1.5707945" effort="1" velocity="1" />
-        <hardware>
-            <motorType>None</motorType>
-            <motorDirection>1</motorDirection>
-            <armature>0</armature>
-        </hardware>
-    </joint>
-    <joint name="left_elbow_pitch_joint" type="revolute">
-        <parent link="left_shoulder_yaw_link" />
-        <child link="left_elbow_pitch_link" />
-        <origin xyz="-0.0800000025 0.02048037438 0.02003692937" rpy="-0.2962759628 -0.3299797087 -0.8151948384" />
-        <axis xyz="0 0 1" />
-        <limit lower="-2.356198" upper="0" effort="1" velocity="1" />
-        <hardware>
-            <motorType>None</motorType>
-            <motorDirection>1</motorDirection>
-            <armature>0</armature>
-        </hardware>
-    </joint>
-    <joint name="left_shoulder_yaw_joint" type="revolute">
-        <parent link="left_shoulder_roll_link" />
-        <child link="left_shoulder_yaw_link" />
-        <origin xyz="0.1148822482 -0.02709980309 -0.03734592284" rpy="-2.701771727 -0.3143027 -3.14158898" />
-        <axis xyz="1 0 0" />
-        <limit lower="-1.5708" upper="1.5708" effort="1" velocity="1" />
-        <hardware>
-            <motorType>None</motorType>
-            <motorDirection>1</motorDirection>
-            <armature>0</armature>
-        </hardware>
-    </joint>
-    <joint name="left_shoulder_roll_joint" type="revolute">
-        <parent link="left_shoulder_pitch_link" />
-        <child link="left_shoulder_roll_link" />
-        <origin xyz="-0.04100000351 0.02565540881 -0.007919662552" rpy="-2.8052323666 0.4653133292 -2.9859660904" />
-        <axis xyz="0 1 0" />
-        <limit lower="-1.57079475" upper="1.91986025" effort="1" velocity="1" />
-        <hardware>
-            <motorType>None</motorType>
-            <motorDirection>1</motorDirection>
-            <armature>0</armature>
-        </hardware>
-    </joint>
-    <joint name="left_shoulder_pitch_joint" type="revolute">
+            <motorDirection>-1</motorDirection>
+            <armature>0</armature>
+        </hardware>
+    </joint>
+    <joint name="right_shoulder_pitch" type="revolute">
         <parent link="world_root" />
-        <child link="left_shoulder_pitch_link" />
-        <origin xyz="0.04962222198 -0.007996932602 0.7928799915" rpy="0.2994274351 0.1745330072 -3.141587582" />
+        <child link="right_shoulder_pitch_link" />
+        <origin xyz="-0.04962609453 -0.007796944815 0.7928799997" rpy="-0.2594571717 -0.1745330458 3.141587621" />
         <axis xyz="-1 0 0" />
         <limit lower="-3.1415916" upper="0.7853984" effort="1" velocity="1" />
@@ -550,5 +575,65 @@
         </hardware>
     </joint>
-    <joint name="right_wrist_pitch_joint" type="revolute">
+    <joint name="right_shoulder_roll" type="revolute">
+        <parent link="right_shoulder_pitch_link" />
+        <child link="right_shoulder_roll_link" />
+        <origin xyz="0.04099980899 0.02527477392 0.006709218258" rpy="0.3501154544 0.7257811284 0.2377861735" />
+        <axis xyz="0 1 0" />
+        <limit lower="-1.91986025" upper="1.57079475" effort="1" velocity="1" />
+        <hardware>
+            <motorType>None</motorType>
+            <motorDirection>-1</motorDirection>
+            <armature>0</armature>
+        </hardware>
+    </joint>
+    <joint name="right_shoulder_yaw" type="revolute">
+        <parent link="right_shoulder_roll_link" />
+        <child link="right_shoulder_yaw_link" />
+        <origin xyz="0.1008846481 -0.02639984048 0.06644494687" rpy="1.55277638 -0.5824100464 3.673220854e-06" />
+        <axis xyz="-1 0 0" />
+        <limit lower="-1.5707972" upper="1.5707972" effort="1" velocity="1" />
+        <hardware>
+            <motorType>None</motorType>
+            <motorDirection>1</motorDirection>
+            <armature>0</armature>
+        </hardware>
+    </joint>
+    <joint name="right_elbow_pitch" type="revolute">
+        <parent link="right_shoulder_yaw_link" />
+        <child link="right_elbow_pitch_link" />
+        <origin xyz="0.08000000295 0.0270258376 -0.009514478403" rpy="-1.552756021 0.04712209601 0.0008482378368" />
+        <axis xyz="0 0 1" />
+        <limit lower="0" upper="2.356199" effort="1" velocity="1" />
+        <hardware>
+            <motorType>None</motorType>
+            <motorDirection>-1</motorDirection>
+            <armature>0</armature>
+        </hardware>
+    </joint>
+    <joint name="right_wrist_yaw" type="revolute">
+        <parent link="right_elbow_pitch_link" />
+        <child link="right_wrist_yaw_motor_link" />
+        <origin xyz="0.0634578 -0.0130041 -0.0264" rpy="3.1415913 5.5e-06 -1.6179277" />
+        <axis xyz="0 1 0" />
+        <limit lower="-1.5707955" upper="1.5707955" effort="1" velocity="1" />
+        <hardware>
+            <motorType>None</motorType>
+            <motorDirection>1</motorDirection>
+            <armature>0</armature>
+        </hardware>
+    </joint>
+    <joint name="right_wrist_roll" type="revolute">
+        <parent link="right_wrist_yaw_motor_link" />
+        <child link="right_wrist_roll_motor_link" />
+        <origin xyz="-4.077257665e-07 -0.137 -0.026" rpy="1.57079999 2.727450251e-07 -1.645121" />
+        <axis xyz="0 1 0" />
+        <limit lower="-0.698132" upper="0.698132" effort="1" velocity="1" />
+        <hardware>
+            <motorType>None</motorType>
+            <motorDirection>1</motorDirection>
+            <armature>0</armature>
+        </hardware>
+    </joint>
+    <joint name="right_wrist_pitch" type="revolute">
         <parent link="right_wrist_roll_motor_link" />
         <child link="right_wrist_pitch_link" />
@@ -558,84 +643,24 @@
         <hardware>
             <motorType>None</motorType>
-            <motorDirection>1</motorDirection>
-            <armature>0</armature>
-        </hardware>
-    </joint>
-    <joint name="right_wrist_roll_joint" type="revolute">
-        <parent link="right_wrist_yaw_motor_link" />
-        <child link="right_wrist_roll_motor_link" />
-        <origin xyz="-4.077257665e-07 -0.137 -0.026" rpy="1.57079999 2.727450251e-07 -1.645121" />
-        <axis xyz="0 1 0" />
-        <limit lower="-0.698132" upper="0.698132" effort="1" velocity="1" />
-        <hardware>
-            <motorType>None</motorType>
             <motorDirection>-1</motorDirection>
             <armature>0</armature>
         </hardware>
     </joint>
-    <joint name="right_wrist_yaw_joint" type="revolute">
-        <parent link="right_elbow_pitch_link" />
-        <child link="right_wrist_yaw_motor_link" />
-        <origin xyz="0.0634578 -0.0130041 -0.0264" rpy="3.1415913 5.5e-06 -1.6179277" />
-        <axis xyz="0 1 0" />
-        <limit lower="-1.5707955" upper="1.5707955" effort="1" velocity="1" />
-        <hardware>
-            <motorType>None</motorType>
-            <motorDirection>-1</motorDirection>
-            <armature>0</armature>
-        </hardware>
-    </joint>
-    <joint name="right_elbow_pitch_joint" type="revolute">
-        <parent link="right_shoulder_yaw_link" />
-        <child link="right_elbow_pitch_link" />
-        <origin xyz="0.08000000295 0.0270258376 -0.009514478403" rpy="-1.552756021 0.04712209601 0.0008482378368" />
-        <axis xyz="0 0 -1" />
-        <limit lower="-2.356199" upper="0" effort="1" velocity="1" />
-        <hardware>
-            <motorType>None</motorType>
-            <motorDirection>-1</motorDirection>
-            <armature>0</armature>
-        </hardware>
-    </joint>
-    <joint name="right_shoulder_yaw_joint" type="revolute">
-        <parent link="right_shoulder_roll_link" />
-        <child link="right_shoulder_yaw_link" />
-        <origin xyz="0.1008846481 -0.02639984048 0.06644494687" rpy="1.55277638 -0.5824100464 3.673220854e-06" />
-        <axis xyz="-1 0 0" />
-        <limit lower="-1.5707972" upper="1.5707972" effort="1" velocity="1" />
-        <hardware>
-            <motorType>None</motorType>
-            <motorDirection>-1</motorDirection>
-            <armature>0</armature>
-        </hardware>
-    </joint>
-    <joint name="right_shoulder_roll_joint" type="revolute">
-        <parent link="right_shoulder_pitch_link" />
-        <child link="right_shoulder_roll_link" />
-        <origin xyz="0.04099980899 0.02527477392 0.006709218258" rpy="0.3501154544 0.7257811284 0.2377861735" />
-        <axis xyz="0 1 0" />
-        <limit lower="-1.91986025" upper="1.57079475" effort="1" velocity="1" />
-        <hardware>
-            <motorType>None</motorType>
-            <motorDirection>1</motorDirection>
-            <armature>0</armature>
-        </hardware>
-    </joint>
-    <joint name="right_shoulder_pitch_joint" type="revolute">
-        <parent link="world_root" />
-        <child link="right_shoulder_pitch_link" />
-        <origin xyz="-0.04962609453 -0.007796944815 0.7928799997" rpy="-0.2594571717 -0.1745330458 3.141587621" />
-        <axis xyz="-1 0 0" />
-        <limit lower="-3.1415916" upper="0.7853984" effort="1" velocity="1" />
-        <hardware>
-            <motorType>None</motorType>
-            <motorDirection>-1</motorDirection>
-            <armature>0</armature>
-        </hardware>
-    </joint>
-    <joint name="left_gripper_joint" type="prismatic">
+    <joint name="left_gripper" type="prismatic">
         <parent link="left_wrist_pitch_link" />
         <child link="left_gripper_finger_left_link" />
         <origin xyz="0.1040961904 -0.04585909073 -0.01258790935" rpy="1.5708 -0.0698132 0.845028" />
+        <axis xyz="1 0 0" />
+        <limit lower="0" upper="0.047" effort="1" velocity="1" />
+        <hardware>
+            <motorType>None</motorType>
+            <motorDirection>1</motorDirection>
+            <armature>0</armature>
+        </hardware>
+    </joint>
+    <joint name="right_gripper" type="prismatic">
+        <parent link="right_wrist_pitch_link" />
+        <child link="right_gripper_finger_left_link" />
+        <origin xyz="0.113421574 -0.009254971529 -0.01265282701" rpy="1.5708 -0.0698132 1.17725" />
         <axis xyz="1 0 0" />
         <limit lower="0" upper="0.047" effort="1" velocity="1" />
@@ -657,17 +682,5 @@
             <armature>0</armature>
         </hardware>
-        <mimic joint="left_gripper_joint" multiplier="1" offset="0" />
-    </joint>
-    <joint name="right_gripper_joint" type="prismatic">
-        <parent link="right_wrist_pitch_link" />
-        <child link="right_gripper_finger_left_link" />
-        <origin xyz="0.113421574 -0.009254971529 -0.01265282701" rpy="1.5708 -0.0698132 1.17725" />
-        <axis xyz="1 0 0" />
-        <limit lower="0" upper="0.047" effort="1" velocity="1" />
-        <hardware>
-            <motorType>None</motorType>
-            <motorDirection>1</motorDirection>
-            <armature>0</armature>
-        </hardware>
+        <mimic joint="left_gripper" multiplier="1" offset="0" />
     </joint>
     <joint name="right_gripper_passive_joint" type="prismatic">
@@ -682,5 +695,5 @@
             <armature>0</armature>
         </hardware>
-        <mimic joint="right_gripper_joint" multiplier="1" offset="0" />
+        <mimic joint="right_gripper" multiplier="1" offset="0" />
     </joint>
     <joint name="head_camera_joint" type="fixed">
@@ -709,3 +722,13 @@
         <origin xyz="0.1551621984 -0.06441037825 -0.01860434352" rpy="1.5708 -0.0698132 1.17725" />
     </joint>
+    <xacro:if value="$(arg emit_ros2_control)">
+        <xacro:lite_ros2_control
+            name="LiteSystem"
+            use_fake_hardware="$(arg use_fake_hardware)"
+            use_sim="$(arg use_sim)"
+            mode="$(arg mode)"
+            can_interface_left="$(arg can_interface_left)"
+            can_interface_right="$(arg can_interface_right)"
+            calibration_file="$(arg calibration_file)"/>
+    </xacro:if>
 </robot>

Commit message: fix: keep default xacro studio-safe

File: urdf/lite.urdf.xacro (robot description, xacro)
@@ -6,5 +6,5 @@
       and optional ros2_control metadata follow lite_urdf.
     -->
-    <xacro:arg name="emit_ros2_control" default="true"/>
+    <xacro:arg name="emit_ros2_control" default="false"/>
     <xacro:arg name="use_fake_hardware" default="true"/>
     <xacro:arg name="use_sim" default="false"/>
@@ -441,4 +441,10 @@
             <geometry>
                 <cylinder radius="0.054721" length="0.209443" />
+            </geometry>
+        </collision>
+        <collision>
+            <origin xyz="-0.0000037 -0.006508 0.952301" rpy="0 0 0" />
+            <geometry>
+                <box size="0.168 0.09 0.16" />
             </geometry>
         </collision>
